File: pcb/pcb/pcb.kicad_pcb (KiCad board)
At the start: 2 copper layers, 100 x 80 mm, 46 parts, among them J1 Conn_01x07, J10 Barrel_Jack, J11 Conn_01x34, J12 Conn_01x12, J13 Conn_01x03, J14 DIN-5_180degree, J15 DIN-5_180degree, J2 Conn_01x07, J3 Conn_01x07, J4 Conn_01x07, J5 Conn_01x07, J6 Conn_01x07, J7 Conn_01x07, J8 Conn_01x07, J9 Conn_01x07, SW1 SW_Push, U1 74HC595, U2 6N137, U3 MCP4811, U4 LM324

Commit message: Maybe finished PCB layout
Parts:
- removed A1: DD39AJPA, footprints:DD39AJPA
- removed REF** (x2): MountingHole_3.2mm_M3_DIN965, MountingHole:MountingHole_3.2mm_M3_DIN965
- added J101: Conn_01x02, Connector_JST:JST_XH_B2B-XH-A_1x02_P2.50mm_Vertical, F.Cu at (270.4, 29.3)
- added J102: Conn_01x03, Connector_JST:JST_XH_B3B-XH-A_1x03_P2.50mm_Vertical, F.Cu at (271.1, 36.9)
- added JP101: Jumper_3_Bridged12, footprints:SolderDipJumper3alt, F.Cu at (279.3, 45.7)
- added U101: do not equip, Package_TO_SOT_THT:TO-220-3_Horizontal_TabDown, F.Cu at (267.9, 70.9)
- added hole1: MountingHole_3.2mm_M3_DIN965, MountingHole:MountingHole_3.2mm_M3_DIN965, F.Cu at (184.8, 29.5)
- added hole2 (x2): MountingHole_3.2mm_M3_DIN965, MountingHole:MountingHole_3.2mm_M3_DIN965, F.Cu at (278.8, 29.5)
- R1, R10, R11, R2, R3, R4, R5, R6, R7, R8, R9: moved to B.Cu
- U4: value LM324 -> LM358; footprint Package_DIP:DIP-14_W7.62mm -> Package_DIP:DIP-8_W7.62mm
- moved JP3 58.8 mm to (270.2, 45.8)
- moved JP1 48.7 mm to (273.9, 45.8), turned to 90 degrees
- moved JP2 42.9 mm to (266.4, 45.8), turned to 90 degrees
- moved SW1 33.9 mm to (232.3, 50.5)
- moved R4 33.1 mm to (217.9, 22.7), turned to 90 degrees
- moved NT1 28.8 mm to (268.9, 20.1)
- moved U2 27.2 mm to (238.9, 33.2), turned to 270 degrees
- moved U3 20.3 mm to (227.9, 33.2), turned to 270 degrees
- moved R11 15.1 mm to (222.7, 47.2), turned to 90 degrees
- moved JP4 15.0 mm to (235.7, 45.3)
- moved R3 14.0 mm to (207.2, 22.8), turned to 270 degrees
- moved R9 13.5 mm to (227.7, 47.3), turned to 90 degrees
- moved R10 12.1 mm to (225.2, 47.2), turned to 270 degrees
- moved R8 11.7 mm to (209.4, 22.8), turned to 270 degrees
- moved R2 10.3 mm to (271.7, 39.5), turned to 180 degrees
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- renumbered REF** to hole1, REF** to hole2, REF** to hole3, REF** to hole4
Connections:
- A2 pad 5V: (no net) -> Net-(A2-Pad5V)
- R11 pad 1: GND -> GNDA
- U3 pad 5: GND -> GNDA
- U3 pad 7: GND -> GNDA
- U4 pad 4: +15V -> -15V
- U4 pad 5: (no net) -> GNDA
- U4 pad 6: (no net) -> Net-(U4-Pad6)
- U4 pad 7: (no net) -> Net-(U4-Pad6)
- U4 pad 8: (no net) -> +15V
Routing:
- net GND: track 0.00 -> 314.6 mm
- net VCC: track 0.00 -> 263.4 mm
- net sck: track 0.00 -> 158.8 mm
- net sda: track 0.00 -> 152.6 mm
- net Net-(A2-PadPA7): track 0.00 -> 139.6 mm
- net GNDA: track 0.00 -> 137.2 mm, vias 0 -> 1
- net +15V: track 0.00 -> 114.1 mm
- net -15V: track 0.00 -> 95.1 mm, vias 0 -> 1
- net Net-(JP2-Pad2): track 0.00 -> 93.7 mm
- net Net-(A2-PadPB1): track 0.00 -> 88.7 mm, vias 0 -> 1
- net Net-(A2-PadPB0): track 0.00 -> 85.1 mm, vias 0 -> 1
- net Net-(A2-PadPA5): track 0.00 -> 83.3 mm, vias 0 -> 1
- net Net-(A2-PadPA6): track 0.00 -> 81.3 mm, vias 0 -> 1
- net /fd0: track 0.00 -> 80.4 mm
- net /fd1: track 0.00 -> 75.3 mm, vias 0 -> 1
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- added copper zone on B.Cu, net GND
- added copper zone on F.Cu, net GND
- added copper zone on B.Cu, net GNDA
- added copper zone on F.Cu, net GNDA
Other:
- board size 100 x 80 mm -> 100 x 80.8 mm

Commit message: silkscreen
Parts:
- removed the hole2 at (278.8, 29.5) (x2)
- added hole2: MountingHole_3.2mm_M3_DIN965, MountingHole:MountingHole_3.2mm_M3_DIN965, F.Cu at (278.8, 29.5)
- renumbered J102 to J16, J101 to J17, JP101 to JP5, U101 to U5
Routing:
- net GND: track 314.6 -> 394.3 mm, vias 0 -> 7
Other:
- board text added: "5V selection"
- board text added: "JLCJLCJLCJLC"
- board text added: "JP1,2,3"
- board text added: "JP4"
- board text added: "MCP4811"
- board text added: "MCP4822"
- board text added: "MIDI in"
- board text added: "MIDI out"
- board text added: "bl** pill"
- board text added: "black pill"
- board text added: "blue pill"
- board text added: "bluepill / blackpill"
- board text added: "via U5"

Commit message: fix hardware bug
Parts:
- added R12: 10k, Resistor_SMD:R_0805_2012Metric, B.Cu at (214.5, 62.3)
- added R13: 10k, Resistor_SMD:R_0805_2012Metric, B.Cu at (212.3, 62.3)
- added R14: 10k, Resistor_SMD:R_0805_2012Metric, B.Cu at (210.0, 62.3)
- added R15: 10k, Resistor_SMD:R_0805_2012Metric, B.Cu at (207.8, 62.3)
- added R16: 10k, Resistor_SMD:R_0805_2012Metric, B.Cu at (205.5, 62.3)
- added R17: 10k, Resistor_SMD:R_0805_2012Metric, B.Cu at (214.5, 58.8)
- added R18: 10k, Resistor_SMD:R_0805_2012Metric, B.Cu at (212.3, 58.8)
- added R19: 10k, Resistor_SMD:R_0805_2012Metric, B.Cu at (210.0, 58.8)
- added R20: 10k, Resistor_SMD:R_0805_2012Metric, B.Cu at (207.8, 58.8)
- added R21: 10k, Resistor_SMD:R_0805_2012Metric, B.Cu at (205.5, 58.8)
Connections:
- J11 pad 30: Net-(A2-PadPB1) -> Net-(J11-Pad30)
- J11 pad 31: Net-(A2-PadPB0) -> Net-(J11-Pad31)
- J11 pad 32: Net-(A2-PadPA7) -> Net-(J11-Pad32)
- J11 pad 33: Net-(A2-PadPA6) -> Net-(J11-Pad33)
- J11 pad 34: Net-(A2-PadPA5) -> Net-(J11-Pad34)
Routing:
- net GND: track 394.3 -> 345.0 mm, vias 7 -> 3
- net Net-(J11-Pad34): track 0.00 -> 28.0 mm
- net Net-(A2-PadPA5): track 83.3 -> 57.5 mm, vias 1 -> 2
- net Net-(J11-Pad33): track 0.00 -> 22.8 mm
- net Net-(J11-Pad32): track 0.00 -> 22.5 mm
- net Net-(A2-PadPA6): track 81.3 -> 60.8 mm, vias 1 -> 2
- net Net-(J11-Pad31): track 0.00 -> 17.2 mm
- net Net-(J11-Pad30): track 0.00 -> 17.0 mm
- net GNDA: track 137.2 -> 153.1 mm, vias 1 -> 2
- net Net-(A2-PadPB0): track 85.1 -> 70.1 mm, vias 1 -> 2
- net Net-(A2-PadPA7): track 139.6 -> 125.8 mm, vias 0 -> 3
- net Net-(A2-PadPB1): track 88.7 -> 75.1 mm, vias 1 -> 2
- net +15V: track 114.1 -> 107.9 mm
