File: pcb/pcb/pcb.sch (KiCad schematic (older format))
At the start: 40 parts, among them J102 Barrel_Jack, J103 Conn_01x07, J105 Conn_01x07, J106 Conn_01x07, J107 Conn_01x07, J108 Conn_01x07, J109 Conn_01x07, J11 Conn_01x34, J111 Conn_01x07, J112 Conn_01x07, J113 Conn_01x07, J12 Conn_01x12, J13 Conn_01x03, J14 DIN-5_180degree, J15 DIN-5_180degree, SW1 SW_Push, U1 74HC595, U2 6N137, U3 MCP4811, U4 LM324

Commit message: pcb++
Parts:
- J13: footprint Connector_JST:JST_XH_B7B-XH-A_1x07_P2.50mm_Vertical -> Connector_PinHeader_2.54mm:PinHeader_1x03_P2.54mm_Horizontal
- renumbered A101 to A1, J103 to J1, J102 to J10, J105 to J2, J106 to J3, J107 to J4, J108 to J5, J109 to J6, J111 to J7, J112 to J8, J113 to J9, R101 to R1, R102 to R2
Other:
- moved on the sheet: A1, J1, J10, J2, J3, J4, J5, J6, J7, J8, J9, R1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

Commit message: Maybe finished PCB layout
Parts:
- removed A1: DD39AJPA, footprints:DD39AJPA, symbol bluepill:DD39AJPA
- removed U4: LM324, Package_DIP:DIP-14_W7.62mm, symbol Amplifier_Operational:LM324
- added J101: Conn_01x02, Connector_JST:JST_XH_B2B-XH-A_1x02_P2.50mm_Vertical, symbol Connector_Generic:Conn_01x02
- added J102: Conn_01x03, Connector_JST:JST_XH_B3B-XH-A_1x03_P2.50mm_Vertical, symbol Connector_Generic:Conn_01x03
- added JP101: Jumper_3_Bridged12, footprints:SolderDipJumper3alt, symbol Jumper:Jumper_3_Bridged12
- added U101: do not equip, Package_TO_SOT_THT:TO-220-3_Horizontal_TabDown, symbol Regulator_Linear:LM7805_TO220
- added U4: LM358, Package_DIP:DIP-8_W7.62mm, symbol Amplifier_Operational:LM358
Connections:
- net +15V: now also J102.3 (Pin_3), U4.8 (V+)
- net +5V: now also JP101.2 (C)
- net +VDC: now also J101.1 (Pin_1), U101.1 (VI)
- net -15V: now also J102.1 (Pin_1), U4.4 (V-)
- net GND: now also U101.2 (GND); no longer R11.1, U3.5 (~LDAC), U3.7 (Vss)
- net GNDA: now also R11.1, U3.5 (~LDAC), U3.7 (Vss), J102.2 (Pin_2), U4.5 (+)
- net GNDPWR: now also J101.2 (Pin_2)
- net dac_out: now also U4.1
- net at A2.5V: now also JP101.1 (A)
- net at U3.8 (Vout): now also U4.3 (+)
- net at R10.1, R11.2: now also U4.2 (-)
- new net: JP101.3 (B), U101.3 (VO)
- new net: U4.6 (-), U4.7
- no-connect marks 12 -> 11
Changed lines of the file:
@@
 	7200 2575 8100 2575
-$Comp
-L power:GND #PWR047
-U 1 1 60F1F258
-P 8100 2575
-F 0 "#PWR047" H 8100 2325 50  0001 C CNN
-F 1 "GND" H 8105 2402 50  0000 C CNN
-F 2 "" H 8100 2575 50  0001 C CNN
-F 3 "" H 8100 2575 50  0001 C CNN
-	1    8100 2575
-	1    0    0    -1
-$EndComp
-Connection ~ 8100 2575
 $Comp
 L power:VCC #PWR046
@@
 	5825 2875 5825 3375
 $Comp
-L Amplifier_Operational:LM324 U4
-U 1 1 60F5EE6A
-P 9325 1725
-F 0 "U4" H 9400 1925 50  0000 C CNN
-F 1 "LM324" H 9425 1575 50  0000 C CNN
-F 2 "Package_DIP:DIP-14_W7.62mm" H 9275 1825 50  0001 C CNN
-F 3 "http://www.ti.com/lit/ds/symlink/lm2902-n.pdf" H 9375 1925 50  0001 C CNN
-	1    9325 1725
-	1    0    0    -1
-$EndComp
-$Comp
-L Amplifier_Operational:LM324 U4
-U 5 1 60F617A5
-P 9325 1725
-F 0 "U4" H 9283 1725 50  0001 L CNN
-F 1 "LM324" H 9283 1680 50  0001 L CNN
-F 2 "Package_DIP:DIP-14_W7.62mm" H 9275 1825 50  0001 C CNN
-F 3 "http://www.ti.com/lit/ds/symlink/lm2902-n.pdf" H 9375 1925 50  0001 C CNN
-	5    9325 1725
-	1    0    0    -1
-$EndComp
-$Comp
 L power:+15V #PWR049
 U 1 1 60F64F72
@@
 	1    0    0    -1
 $EndComp
-NoConn ~ 4100 2225
 NoConn ~ 3800 2225
 $Comp
@@
 Wire Wire Line
 	9625 2375 9625 2325
-$Comp
-L power:GND #PWR051
-U 1 1 612AA6BC
-P 9625 2675
-F 0 "#PWR051" H 9625 2425 50  0001 C CNN
-F 1 "GND" H 9630 2502 50  0000 C CNN
-F 2 "" H 9625 2675 50  0001 C CNN
-F 3 "" H 9625 2675 50  0001 C CNN
-	1    9625 2675
-	1    0    0    -1
-$EndComp
 Wire Wire Line
 	9625 2325 9025 2325
@@
 	1375 7425 1600 7425
 $Comp
-L bluepill:DD39AJPA A1
-U 1 1 614B1B14
-P 2150 7325
-F 0 "A1" H 2125 7650 50  0000 C CNN
-F 1 "DD39AJPA" H 2125 7559 50  0000 C CNN
-F 2 "footprints:DD39AJPA" H 2150 7325 50  0001 C CNN
-F 3 "" H 2150 7325 50  0001 C CNN
-	1    2150 7325
-	1    0    0    -1
-$EndComp
-$Comp
 L power:GNDPWR #PWR020
 U 1 1 614769FE
@@
 	1    0    0    -1
 $EndComp
+$Comp
+L Connector_Generic:Conn_01x02 J101
+U 1 1 60CEB0CE
+P 1800 7275
+F 0 "J101" H 1880 7267 50  0000 L CNN
+F 1 "Conn_01x02" H 1880 7176 50  0000 L CNN
+F 2 "Connector_JST:JST_XH_B2B-XH-A_1x02_P2.50mm_Vertical" H 1800 7275 50  0001 C CNN
+F 3 "~" H 1800 7275 50  0001 C CNN
+	1    1800 7275
+	1    0    0    -1
+$EndComp
+$Comp
+L Connector_Generic:Conn_01x03 J102
+U 1 1 60CEE5AD
+P 2450 7325
+F 0 "J102" H 2368 7000 50  0000 C CNN
+F 1 "Conn_01x03" H 2368 7091 50  0000 C CNN
+F 2 "Connector_JST:JST_XH_B3B-XH-A_1x03_P2.50mm_Vertical" H 2450 7325 50  0001 C CNN
+F 3 "~" H 2450 7325 50  0001 C CNN
+	1    2450 7325
+	-1   0    0    1
+$EndComp
+$Comp
+L Regulator_Linear:LM7805_TO220 U101
+U 1 1 60D0B8E5
+P 3300 1850
+F 0 "U101" H 3300 2092 50  0000 C CNN
+F 1 "do not equip" H 3300 2001 50  0000 C CNN
+F 2 "Package_TO_SOT_THT:TO-220-3_Horizontal_TabDown" H 3300 2075 50  0001 C CIN
+F 3 "https://www.onsemi.cn/PowerSolutions/document/MC7800-D.PDF" H 3300 1800 50  0001 C CNN
+	1    3300 1850
+	1    0    0    -1
+$EndComp
+$Comp
+L power:+VDC #PWR0101
+U 1 1 60D13602
+P 3000 1850
+F 0 "#PWR0101" H 3000 1750 50  0001 C CNN
+F 1 "+VDC" H 3000 2125 50  0000 C CNN
+F 2 "" H 3000 1850 50  0001 C CNN
+F 3 "" H 3000 1850 50  0001 C CNN
+	1    3000 1850
+	1    0    0    -1
+$EndComp
+$Comp
+L power:GND #PWR0102
+U 1 1 60D14706
+P 3300 2150
+F 0 "#PWR0102" H 3300 1900 50  0001 C CNN
+F 1 "GND" H 3350 1975 50  0000 C CNN
+F 2 "" H 3300 2150 50  0001 C CNN
+F 3 "" H 3300 2150 50  0001 C CNN
+	1    3300 2150
+	1    0    0    -1
+$EndComp
+$Comp
+L Jumper:Jumper_3_Bridged12 JP101
+U 1 1 60D1BB6F
+P 3850 1850
+F 0 "JP101" H 3850 1961 50  0000 C CNN
+F 1 "Jumper_3_Bridged12" H 3850 2052 50  0000 C CNN
+F 2 "footprints:SolderDipJumper3alt" H 3850 1850 50  0001 C CNN
+F 3 "~" H 3850 1850 50  0001 C CNN
+	1    3850 1850
+	-1   0    0    1
+$EndComp
+Wire Wire Line
+	4100 1850 4100 2225
+$Comp
+L power:+5V #PWR0103
+U 1 1 60DCE804
+P 3850 1700
+F 0 "#PWR0103" H 3850 1550 50  0001 C CNN
+F 1 "+5V" H 3865 1873 50  0000 C CNN
+F 2 "" H 3850 1700 50  0001 C CNN
+F 3 "" H 3850 1700 50  0001 C CNN
+	1    3850 1700
+	1    0    0    -1
+$EndComp
+$Comp
+L power:GNDA #PWR0104
+U 1 1 60E07F1C
+P 8100 2575
+F 0 "#PWR0104" H 8100 2325 50  0001 C CNN
+F 1 "GNDA" H 8105 2402 50  0000 C CNN
+F 2 "" H 8100 2575 50  0001 C CNN
+F 3 "" H 8100 2575 50  0001 C CNN
+	1    8100 2575
+	1    0    0    -1
+$EndComp
+Connection ~ 8100 2575
+$Comp
+L power:GNDA #PWR0105
+U 1 1 60E0E8CF
+P 9625 2675
+F 0 "#PWR0105" H 9625 2425 50  0001 C CNN
+F 1 "GNDA" H 9630 2502 50  0000 C CNN
+F 2 "" H 9625 2675 50  0001 C CNN
+F 3 "" H 9625 2675 50  0001 C CNN
+	1    9625 2675
+	1    0    0    -1
+$EndComp
+$Comp
+L Amplifier_Operational:LM358 U4
+U 1 1 60E3D864
+P 9325 1725
+F 0 "U4" H 9325 2000 50  0000 C CNN
+F 1 "LM358" H 9325 2001 50  0001 C CNN
+F 2 "Package_DIP:DIP-8_W7.62mm" H 9325 1725 50  0001 C CNN
+F 3 "http://www.ti.com/lit/ds/symlink/lm2904-n.pdf" H 9325 1725 50  0001 C CNN
+	1    9325 1725
+	1    0    0    -1
+$EndComp
+$Comp
+L Amplifier_Operational:LM358 U4
+U 3 1 60E401C0
+P 9325 1725
+F 0 "U4" H 9375 1875 50  0001 L CNN
+F 1 "LM358" H 9250 1725 50  0000 L CNN
+F 2 "Package_DIP:DIP-8_W7.62mm" H 9325 1725 50  0001 C CNN
+F 3 "http://www.ti.com/lit/ds/symlink/lm2904-n.pdf" H 9325 1725 50  0001 C CNN
+	3    9325 1725
+	1    0    0    -1
+$EndComp
+$Comp
+L Amplifier_Operational:LM358 U4
+U 2 1 60E41959
+P 10500 3975
+F 0 "U4" H 10500 4342 50  0000 C CNN
+F 1 "LM358" H 10500 4251 50  0000 C CNN
+F 2 "Package_DIP:DIP-8_W7.62mm" H 10500 3975 50  0001 C CNN
+F 3 "http://www.ti.com/lit/ds/symlink/lm2904-n.pdf" H 10500 3975 50  0001 C CNN
+	2    10500 3975
+	1    0    0    -1
+$EndComp
+Wire Wire Line
+	10200 4075 10200 4250
+Wire Wire Line
+	10200 4250 10800 4250
+Wire Wire Line
+	10800 4250 10800 3975
+$Comp
+L power:GNDA #PWR0106
+U 1 1 60E622F6
+P 10100 3875
+F 0 "#PWR0106" H 10100 3625 50  0001 C CNN
+F 1 "GNDA" H 10105 3702 50  0000 C CNN
+F 2 "" H 10100 3875 50  0001 C CNN
+F 3 "" H 10100 3875 50  0001 C CNN
+	1    10100 3875
+	1    0    0    -1
+$EndComp
+Wire Wire Line
+	10100 3875 10200 3875
 Wire Wire Line
 	4700 2875 5825 2875

Commit message: silkscreen
Parts:
- renumbered J102 to J16, J101 to J17, JP101 to JP5, U101 to U5
Changed lines of the file:
@@
 $EndComp
 $Comp
-L Connector_Generic:Conn_01x02 J101
+L Connector_Generic:Conn_01x02 J17
 U 1 1 60CEB0CE
 P 1800 7275
-F 0 "J101" H 1880 7267 50  0000 L CNN
+F 0 "J17" H 1880 7267 50  0000 L CNN
 F 1 "Conn_01x02" H 1880 7176 50  0000 L CNN
 F 2 "Connector_JST:JST_XH_B2B-XH-A_1x02_P2.50mm_Vertical" H 1800 7275 50  0001 C CNN
@@
 $EndComp
 $Comp
-L Connector_Generic:Conn_01x03 J102
+L Connector_Generic:Conn_01x03 J16
 U 1 1 60CEE5AD
 P 2450 7325
-F 0 "J102" H 2368 7000 50  0000 C CNN
+F 0 "J16" H 2368 7000 50  0000 C CNN
 F 1 "Conn_01x03" H 2368 7091 50  0000 C CNN
 F 2 "Connector_JST:JST_XH_B3B-XH-A_1x03_P2.50mm_Vertical" H 2450 7325 50  0001 C CNN
@@
 	1    2450 7325
 	-1   0    0    1
-$EndComp
-$Comp
-L Regulator_Linear:LM7805_TO220 U101
-U 1 1 60D0B8E5
-P 3300 1850
-F 0 "U101" H 3300 2092 50  0000 C CNN
-F 1 "do not equip" H 3300 2001 50  0000 C CNN
-F 2 "Package_TO_SOT_THT:TO-220-3_Horizontal_TabDown" H 3300 2075 50  0001 C CIN
-F 3 "https://www.onsemi.cn/PowerSolutions/document/MC7800-D.PDF" H 3300 1800 50  0001 C CNN
-	1    3300 1850
-	1    0    0    -1
 $EndComp
 $Comp
@@
 $EndComp
 $Comp
-L Jumper:Jumper_3_Bridged12 JP101
+L Jumper:Jumper_3_Bridged12 JP5
 U 1 1 60D1BB6F
 P 3850 1850
-F 0 "JP101" H 3850 1961 50  0000 C CNN
+F 0 "JP5" H 3850 1961 50  0000 C CNN
 F 1 "Jumper_3_Bridged12" H 3850 2052 50  0000 C CNN
 F 2 "footprints:SolderDipJumper3alt" H 3850 1850 50  0001 C CNN
@@
 Wire Bus Line
 	5050 2575 5050 5225
+$Comp
+L Regulator_Linear:LM7805_TO220 U5
+U 1 1 60D0B8E5
+P 3300 1850
+F 0 "U5" H 3300 2092 50  0000 C CNN
+F 1 "do not equip" H 3300 2001 50  0000 C CNN
+F 2 "Package_TO_SOT_THT:TO-220-3_Horizontal_TabDown" H 3300 2075 50  0001 C CIN
+F 3 "https://www.onsemi.cn/PowerSolutions/document/MC7800-D.PDF" H 3300 1800 50  0001 C CNN
+	1    3300 1850
+	1    0    0    -1
+$EndComp
 $EndSCHEMATC

Commit message: fix hardware bug
Parts:
- added R12, R13, R14, R15, R16, R17, R18, R19, R20, R21: 10k, Resistor_SMD:R_0805_2012Metric, symbol Device:R
Connections:
- net GNDA: now also R17.2, R18.2, R19.2, R20.2, R21.2
- net at J11.30 (Pin_30): now also R16.1; no longer A2.PB1
- net at J11.31 (Pin_31): now also R15.1; no longer A2.PB0
- net at J11.32 (Pin_32): now also R14.1; no longer A2.PA7
- net at J11.33 (Pin_33): now also R13.1; no longer A2.PA6
- net at J11.34 (Pin_34): now also R12.1; no longer A2.PA5
- new net: A2.PA5, R12.2, R17.1
- new net: A2.PA6, R13.2, R18.1
- new net: A2.PA7, R14.2, R19.1
- new net: A2.PB0, R15.2, R20.1
- new net: A2.PB1, R16.2, R21.1
Changed lines of the file:
@@
 Title ""
 Date ""
-Rev ""
+Rev "02"
 Comp ""
 Comment1 ""
@@
 	1    0    0    -1
 $EndComp
-Wire Wire Line
-	925  1925 2225 1925
-Wire Wire Line
-	925  2025 2150 2025
-Wire Wire Line
-	925  2125 2075 2125
-Wire Wire Line
-	925  2225 2000 2225
-Wire Wire Line
-	925  2325 1925 2325
 $Comp
 L Connector_Generic:Conn_01x34 J11
@@
 Note: the connector is reversed
 Wire Wire Line
-	2225 3275 3200 3275
-Wire Wire Line
-	2150 3375 3200 3375
-Wire Wire Line
-	2075 3475 3200 3475
-Wire Wire Line
-	2000 3575 3200 3575
-Wire Wire Line
-	1925 3675 3200 3675
-Wire Wire Line
 	4775 3400 5225 3400
 Wire Wire Line
@@
 $EndComp
 Wire Wire Line
-	2225 1925 2225 3275
-Wire Wire Line
-	2075 2125 2075 3475
-Wire Wire Line
-	2150 2025 2150 3375
-Wire Wire Line
-	2000 2225 2000 3575
-Wire Wire Line
-	1925 2325 1925 3675
-Wire Wire Line
 	2550 2875 3200 2875
 Wire Wire Line
@@
 Wire Wire Line
 	10100 3875 10200 3875
-Wire Wire Line
-	4700 2875 5825 2875
-Wire Bus Line
-	2850 3875 2850 5225
-Wire Bus Line
-	1275 3625 1275 5225
-Wire Bus Line
-	5050 2575 5050 5225
 $Comp
 L Regulator_Linear:LM7805_TO220 U5
@@
 	1    0    0    -1
 $EndComp
+$Comp
+L Device:R R12
+U 1 1 60F9BFE2
+P 1725 1725
+F 0 "R12" V 1775 1975 50  0000 R CNN
+F 1 "10k" V 1725 1650 50  0000 L CNN
+F 2 "Resistor_SMD:R_0805_2012Metric" V 1655 1725 50  0001 C CNN
+F 3 "~" H 1725 1725 50  0001 C CNN
+	1    1725 1725
+	0    -1   -1   0
+$EndComp
+$Comp
+L Device:R R17
+U 1 1 6101BE24
+P 2025 1725
+F 0 "R17" V 2075 1425 50  0000 L CNN
+F 1 "10k" V 2025 1650 50  0000 L CNN
+F 2 "Resistor_SMD:R_0805_2012Metric" V 1955 1725 50  0001 C CNN
+F 3 "~" H 2025 1725 50  0001 C CNN
+	1    2025 1725
+	0    -1   -1   0
+$EndComp
+$Comp
+L Device:R R13
+U 1 1 6103691E
+P 1725 1900
+F 0 "R13" V 1775 2150 50  0000 R CNN
+F 1 "10k" V 1725 1825 50  0000 L CNN
+F 2 "Resistor_SMD:R_0805_2012Metric" V 1655 1900 50  0001 C CNN
+F 3 "~" H 1725 1900 50  0001 C CNN
+	1    1725 1900
+	0    -1   -1   0
+$EndComp
+$Comp
+L Device:R R14
+U 1 1 61041291
+P 1725 2075
+F 0 "R14" V 1775 2325 50  0000 R CNN
+F 1 "10k" V 1725 2000 50  0000 L CNN
+F 2 "Resistor_SMD:R_0805_2012Metric" V 1655 2075 50  0001 C CNN
+F 3 "~" H 1725 2075 50  0001 C CNN
+	1    1725 2075
+	0    -1   -1   0
+$EndComp
+$Comp
+L Device:R R19
+U 1 1 61041297
+P 2025 2075
+F 0 "R19" V 2075 1775 50  0000 L CNN
+F 1 "10k" V 2025 2000 50  0000 L CNN
+F 2 "Resistor_SMD:R_0805_2012Metric" V 1955 2075 50  0001 C CNN
+F 3 "~" H 2025 2075 50  0001 C CNN
+	1    2025 2075
+	0    -1   -1   0
+$EndComp
+$Comp
+L Device:R R15
+U 1 1 6104BBEE
+P 1725 2250
+F 0 "R15" V 1775 2500 50  0000 R CNN
+F 1 "10k" V 1725 2175 50  0000 L CNN
+F 2 "Resistor_SMD:R_0805_2012Metric" V 1655 2250 50  0001 C CNN
+F 3 "~" H 1725 2250 50  0001 C CNN
+	1    1725 2250
+	0    -1   -1   0
+$EndComp
+$Comp
+L Device:R R20
+U 1 1 6104BBF4
+P 2025 2250
+F 0 "R20" V 2075 1950 50  0000 L CNN
+F 1 "10k" V 2025 2175 50  0000 L CNN
+F 2 "Resistor_SMD:R_0805_2012Metric" V 1955 2250 50  0001 C CNN
+F 3 "~" H 2025 2250 50  0001 C CNN
+	1    2025 2250
+	0    -1   -1   0
+$EndComp
+$Comp
+L Device:R R16
+U 1 1 61056599
+P 1725 2425
+F 0 "R16" V 1775 2675 50  0000 R CNN
+F 1 "10k" V 1725 2350 50  0000 L CNN
+F 2 "Resistor_SMD:R_0805_2012Metric" V 1655 2425 50  0001 C CNN
+F 3 "~" H 1725 2425 50  0001 C CNN
+	1    1725 2425
+	0    -1   -1   0
+$EndComp
+$Comp
+L Device:R R21
+U 1 1 6105659F
+P 2025 2425
+F 0 "R21" V 2075 2125 50  0000 L CNN
+F 1 "10k" V 2025 2350 50  0000 L CNN
+F 2 "Resistor_SMD:R_0805_2012Metric" V 1955 2425 50  0001 C CNN
+F 3 "~" H 2025 2425 50  0001 C CNN
+	1    2025 2425
+	0    -1   -1   0
+$EndComp
+Wire Wire Line
+	925  1925 1100 1925
+Wire Wire Line
+	1100 1925 1100 1725
+Wire Wire Line
+	1100 1725 1575 1725
+Wire Wire Line
+	925  2025 1175 2025
+Wire Wire Line
+	1175 2025 1175 1900
+Wire Wire Line
+	1175 1900 1575 1900
+Wire Wire Line
+	925  2125 1575 2125
+Wire Wire Line
+	1575 2125 1575 2075
+Wire Wire Line
+	925  2225 1575 2225
+Wire Wire Line
+	1575 2225 1575 2250
+Wire Wire Line
+	925  2325 1450 2325
+Wire Wire Line
+	1450 2325 1450 2425
+Wire Wire Line
+	1450 2425 1575 2425
+Wire Wire Line
+	2175 1725 2175 1900
+Connection ~ 2175 1900
+Wire Wire Line
+	2175 1900 2175 2075
+Connection ~ 2175 2075
+Wire Wire Line
+	2175 2075 2175 2250
+Connection ~ 2175 2250
+Wire Wire Line
+	2175 2250 2175 2425
+Connection ~ 2175 2425
+Wire Wire Line
+	2175 2425 2175 2550
+Wire Wire Line
+	1875 1725 1875 1800
+Wire Wire Line
+	1875 1800 2850 1800
+Wire Wire Line
+	2850 1800 2850 3275
+Wire Wire Line
+	2850 3275 3200 3275
+Connection ~ 1875 1725
+Wire Wire Line
+	3200 3375 2800 3375
+Wire Wire Line
+	2800 3375 2800 1975
+Wire Wire Line
+	2800 1975 1875 1975
+Wire Wire Line
+	1875 1975 1875 1900
+Connection ~ 1875 1900
+Wire Wire Line
+	1875 2075 1875 2175
+Wire Wire Line
+	1875 2175 2750 2175
+Wire Wire Line
+	2750 2175 2750 3475
+Wire Wire Line
+	2750 3475 3200 3475
+Connection ~ 1875 2075
+Wire Wire Line
+	2700 2325 1875 2325
+Wire Wire Line
+	1875 2325 1875 2250
+Connection ~ 1875 2250
+Wire Wire Line
+	1875 2425 1875 2500
+Wire Wire Line
+	1875 2500 2650 2500
+Wire Wire Line
+	2650 2500 2650 3675
+Wire Wire Line
+	2650 3675 3200 3675
+Connection ~ 1875 2425
+Wire Wire Line
+	2700 3575 3200 3575
+Wire Wire Line
+	2700 2325 2700 3575
+Wire Wire Line
+	4700 2875 5825 2875
+Wire Bus Line
+	2850 3875 2850 5225
+Wire Bus Line
+	1275 3625 1275 5225
+Wire Bus Line
+	5050 2575 5050 5225
+$Comp
+L Device:R R18
+U 1 1 61036924
+P 2025 1900
+F 0 "R18" V 2075 1600 50  0000 L CNN
+F 1 "10k" V 2025 1825 50  0000 L CNN
+F 2 "Resistor_SMD:R_0805_2012Metric" V 1955 1900 50  0001 C CNN
+F 3 "~" H 2025 1900 50  0001 C CNN
+	1    2025 1900
+	0    -1   -1   0
+$EndComp
+$Comp
+L power:GNDA #PWR0107
+U 1 1 6115B9F4
+P 2175 2550
+F 0 "#PWR0107" H 2175 2300 50  0001 C CNN
+F 1 "GNDA" H 2350 2550 50  0000 C CNN
+F 2 "" H 2175 2550 50  0001 C CNN
+F 3 "" H 2175 2550 50  0001 C CNN
+	1    2175 2550
+	1    0    0    -1
+$EndComp
